File: IsoPCB/IsoPCB.kicad_sch (KiCad schematic)
At the start: 0 parts

Commit message: Bauteile eingepflegt und Schaltplan erstellt
Parts:
- added J1: Conn_02x02_Counter_Clockwise, Connector_PinHeader_2.54mm:PinHeader_2x02_P2.54mm_Horizontal, symbol Connector_Generic:Conn_02x02_Counter_Clockwise
- added J2: Conn_02x02_Counter_Clockwise, Connector_PinSocket_2.54mm:PinSocket_2x02_P2.54mm_Horizontal, symbol Connector_Generic:Conn_02x02_Counter_Clockwise
Connections:
- new net PWM_iso/12V: J1.1 (Pin_1)
- new net PWM_iso/GND: J1.2 (Pin_2)
- new net PWM_iso/PWM_IN: J1.4 (Pin_4)
- new net PWM_iso/PWM_OUT: J2.4 (Pin_4)
- new net PWM_iso/V-_DRIVER: J2.3 (Pin_3)
- new net PowerSupply_iso/GND_Driver: J2.2 (Pin_2)
- new net PowerSupply_iso/V+_Driver: J2.1 (Pin_1)
Other:
- added sheet PWM_iso (PWM_iso.kicad_sch)
- added sheet PowerSupply_iso (PowerSupply_iso.kicad_sch)
- note added: "Mikrocontroller Seite"
- note added: "Treiber Seite"
- company: (none) -> Technische Universität Berlin - Fachgebiet Leistungselektronik
- title: (none) -> Isolierplatine
